Commit message: added mass and inertia to fix pybyllet warnings.

File: robots/hsrb4s.urdf (robot description, URDF)
Before this commit: robot hsrb, 45 links, 44 joints
Links:
- link base_footprint: mass None -> 0.01
- link base_imu_frame: mass None -> 0.0
- link base_range_sensor_link: mass None -> 0.0
- link hand_camera_frame: mass None -> 0.0
- link hand_camera_gazebo_frame: mass None -> 0.0
- link head_center_camera_frame: mass None -> 0.0
- link head_center_camera_gazebo_frame: mass None -> 0.0
- link head_l_stereo_camera_gazebo_frame: mass None -> 0.0
- link head_l_stereo_camera_link: mass None -> 0.0
- link head_r_stereo_camera_gazebo_frame: mass None -> 0.0
- link head_r_stereo_camera_link: mass None -> 0.0
- link head_rgbd_sensor_gazebo_frame: mass None -> 0.0
- link head_rgbd_sensor_link: mass None -> 0.0
- link wrist_ft_sensor_frame: mass None -> 0.0

Commit message: fixed lower and upper.

File: robots/hsrb4s.urdf (robot description, URDF)
Before this commit: robot hsrb, 45 links, 44 joints
Joints:
- joint arm_lift_joint: limit lower=0.0 upper=0.69 effort=100.0 velocity=0.2 -> lower=0.0 upper=0.3 effort=100.0 velocity=0.2
- joint base_roll_joint: limit effort=34.46 velocity=2.5 -> lower=-3.14159 upper=3.14159 effort=34.46 velocity=2.5

Commit message: deleted gazebo tags. deleted all of the hand joints.

File: robots/hsrb4s.urdf (robot description, URDF)
Before this commit: robot hsrb, 45 links, 44 joints
Links:
- removed link hand_camera_frame
- removed link hand_camera_gazebo_frame
- removed link hand_l_distal_link
- removed link hand_l_finger_tip_frame
- removed link hand_l_finger_vacuum_frame
- removed link hand_l_mimic_distal_link
- removed link hand_l_proximal_link
- removed link hand_l_spring_proximal_link
- removed link hand_motor_dummy_link
- removed link hand_palm_link
- removed link hand_r_distal_link
- removed link hand_r_finger_tip_frame
- removed link hand_r_mimic_distal_link
- removed link hand_r_proximal_link
- removed link hand_r_spring_proximal_link
Joints:
- removed joint hand_camera_frame_joint
- removed joint hand_camera_gazebo_frame_joint
- removed joint hand_l_distal_joint
- removed joint hand_l_finger_tip_frame_joint
- removed joint hand_l_finger_vacuum_frame_joint
- removed joint hand_l_mimic_distal_joint
- removed joint hand_l_proximal_joint
- removed joint hand_l_spring_proximal_joint
- removed joint hand_motor_joint
- removed joint hand_palm_joint
- removed joint hand_r_distal_joint
- removed joint hand_r_finger_tip_frame_joint
- removed joint hand_r_mimic_distal_joint
- removed joint hand_r_proximal_joint
- removed joint hand_r_spring_proximal_joint
- joint arm_roll_joint: limit lower=-2.09 upper=3.84 effort=100.0 velocity=2.0 -> lower=-3.14159265359 upper=3.14159265359 effort=100.0 velocity=2.0
- joint base_roll_joint: limit lower=-3.14159 upper=3.14159 effort=34.46 velocity=2.5 -> lower=-3.14159265359 upper=3.14159265359 effort=34.46 velocity=2.5
- joint wrist_flex_joint: limit lower=-1.92 upper=1.22 effort=100.0 velocity=1.5 -> lower=-1.5707963268 upper=1.5707963268 effort=100.0 velocity=1.5
- joint wrist_roll_joint: limit lower=-1.92 upper=3.67 effort=100.0 velocity=1.5 -> lower=-3.14159265359 upper=3.14159265359 effort=100.0 velocity=1.5

Commit message: fixed lower and upper.

File: robots/hsrb4s.urdf (robot description, URDF)
Before this commit: robot hsrb, 30 links, 29 joints
Joints:
- joint head_pan_joint: limit lower=-3.84 upper=1.75 effort=100.0 velocity=1.0 -> lower=-1.5707963268 upper=1.5707963268 effort=100.0 velocity=1.0
- joint head_tilt_joint: limit lower=-1.57 upper=0.52 effort=100.0 velocity=1.0 -> lower=-0.78539816339 upper=0.78539816339 effort=100.0 velocity=1.0

Commit message: fixed lower and upper.

File: robots/hsrb4s.urdf (robot description, URDF)
Before this commit: robot hsrb, 30 links, 29 joints
Joints:
- joint head_pan_joint: limit lower=-1.5707963268 upper=1.5707963268 effort=100.0 velocity=1.0 -> lower=-3.14159265359 upper=3.14159265359 effort=100.0 velocity=1.0
